File: kicad/Projeto_led_natal/Projeto_led_natal-sem_led.kicad_pcb (KiCad board)
At the start: 2 copper layers, 34 parts, among them P1 220K, Q1 BC548, Q2 BC548, Q3 BC548, Q4 BC548, T1 12+12 500mA

Commit message: from note-valmir
Parts:
- moved R1 0.89 mm to (82.5, 101.6)
- moved R2 0.89 mm to (82.5, 94.0)
Routing:
- net Net-(CI-2-THR): track 62.1 -> 51.1 mm
- net GND: track 314.2 -> 310.9 mm
- net Net-(CI-1-OUT): track 90.6 -> 87.6 mm
- net Net-(CI-2-DIS): track 19.9 -> 19.0 mm
Changed lines of the file:
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@@
 	(footprint "Resistor_THT:R_Axial_DIN0204_L3.6mm_D1.6mm_P5.08mm_Vertical"
 		(layer "F.Cu")
-		(at 82.54 94.87 90)
+		(at 82.55 93.98 90)
 		(descr "Resistor, Axial_DIN0204 series, Axial, Vertical, pin pitch=5.08mm, 0.167W, length*diameter=3.6*1.6mm^2, http://cdn-reichelt.de/documents/datenblatt/B400/1_4W%23YAG.pdf")
 		(tags "Resistor Axial_DIN0204 series Axial Vertical pin pitch 5.08mm 0.167W length 3.6mm diameter 1.6mm")
@@
 	(footprint "Resistor_THT:R_Axial_DIN0204_L3.6mm_D1.6mm_P5.08mm_Vertical"
 		(layer "F.Cu")
-		(at 82.54 102.49 90)
+		(at 82.55 101.6 90)
 		(descr "Resistor, Axial_DIN0204 series, Axial, Vertical, pin pitch=5.08mm, 0.167W, length*diameter=3.6*1.6mm^2, http://cdn-reichelt.de/documents/datenblatt/B400/1_4W%23YAG.pdf")
 		(tags "Resistor Axial_DIN0204 series Axial Vertical pin pitch 5.08mm 0.167W length 3.6mm diameter 1.6mm")
@@
 	)
 	(segment
-		(start 96.52 95.25)
-		(end 101.6 95.25)
-		(width 1)
-		(layer "F.Cu")
-		(net 2)
-	)
-	(segment
 		(start 146.05 44.45)
 		(end 146.05 50.8)
@@
 	)
 	(segment
-		(start 146.05 50.8)
-		(end 146.05 57.15)
+		(start 96.52 88.9)
+		(end 96.52 90.17)
 		(width 1)
 		(layer "F.Cu")
@@
 	)
 	(segment
-		(start 88.9 81.28)
-		(end 96.52 88.9)
+		(start 146.05 50.8)
+		(end 146.05 57.15)
 		(width 1)
 		(layer "F.Cu")
@@
 	)
 	(segment
-		(start 96.52 88.9)
-		(end 96.52 95.25)
+		(start 88.9 81.28)
+		(end 96.52 88.9)
 		(width 1)
 		(layer "F.Cu")
@@
 	)
 	(segment
-		(start 93.98 81.28)
-		(end 93.98 78.7)
-		(width 1)
-		(layer "F.Cu")
-		(net 3)
-	)
-	(segment
-		(start 90.52 85.9)
-		(end 81.93 85.9)
+		(start 96.52 90.17)
+		(end 101.6 95.25)
 		(width 1)
 		(layer "F.Cu")
-		(net 3)
+		(net 2)
 	)
 	(segment
-		(start 82.54 89.79)
-		(end 82.47 89.86)
+		(start 91.4 78.7)
+		(end 76.2 78.7)
 		(width 1)
 		(layer "F.Cu")
@@
 	)
 	(segment
-		(start 91.44 88.9)
-		(end 91.44 86.82)
+		(start 83.82 81.28)
+		(end 81.24 78.7)
 		(width 1)
 		(layer "F.Cu")
@@
 	)
 	(segment
-		(start 81.93 85.9)
-		(end 81.93 78.7)
+		(start 93.98 81.28)
+		(end 91.4 78.7)
 		(width 1)
 		(layer "F.Cu")
@@
 	(segment
 		(start 91.44 88.9)
-		(end 91.41 88.87)
-		(width 1)
-		(layer "F.Cu")
-		(net 3)
-	)
-	(segment
-		(start 93.98 78.7)
-		(end 76.2 78.7)
+		(end 83.82 81.28)
 		(width 1)
 		(layer "F.Cu")
@@
 	)
 	(segment
-		(start 82.47 89.86)
-		(end 76.2 89.86)
+		(start 82.55 88.9)
+		(end 76.2 82.55)
 		(width 1)
 		(layer "F.Cu")
@@
 	)
 	(segment
-		(start 91.44 86.82)
-		(end 90.52 85.9)
-		(width 1)
-		(layer "F.Cu")
-		(net 3)
-	)
-	(segment
-		(start 81.24 78.7)
+		(start 76.2 82.55)
 		(end 76.2 78.7)
 		(width 1)
@@
 	)
 	(segment
-		(start 76.2 89.86)
+		(start 81.24 78.7)
 		(end 76.2 78.7)
 		(width 1)
@@
 	)
 	(segment
-		(start 93.98 94.8)
-		(end 93.98 88.9)
-		(width 1)
-		(layer "F.Cu")
-		(net 5)
-	)
-	(segment
-		(start 82.54 94.87)
-		(end 82.54 97.41)
+		(start 82.55 93.98)
+		(end 82.55 96.52)
 		(width 0.2)
 		(layer "F.Cu")
@@
 	)
 	(segment
-		(start 82.54 94.87)
-		(end 82.61 94.8)
+		(start 82.55 93.98)
+		(end 93.98 93.98)
 		(width 1)
 		(layer "F.Cu")
@@
 	)
 	(segment
-		(start 82.61 94.8)
-		(end 93.98 94.8)
+		(start 93.98 93.98)
+		(end 93.98 88.9)
 		(width 1)
 		(layer "F.Cu")
@@
 	)
 	(segment
-		(start 82.83 102.2)
-		(end 99.73 102.2)
+		(start 82.55 101.6)
+		(end 100.33 101.6)
 		(width 1)
 		(layer "F.Cu")
@@
 	)
 	(segment
-		(start 99.73 102.2)
+		(start 100.33 101.6)
 		(end 101.6 100.33)
 		(width 1)
@@
 	)
 	(segment
-		(start 82.54 102.49)
-		(end 82.83 102.2)
-		(width 1)
-		(layer "F.Cu")
-		(net 17)
-	)
-	(segment
 		(start 133.35 82.55)
 		(end 137.16 86.36)
@@
 	)
 	(segment
-		(start 116.9 69.87)
-		(end 116.92 69.85)
-		(width 1)
-		(layer "F.Cu")
-		(net 19)
-	)
-	(segment
 		(start 120.65 71.12)
-		(end 120.65 66.65)
+		(end 120.65 69.7)
 		(width 1)
 		(layer "F.Cu")
@@
 	)
 	(segment
-		(start 139.7 93.98)
-		(end 116.9 93.98)
-		(width 1)
-		(layer "F.Cu")
-		(net 19)
-	)
-	(segment
 		(start 107.95 47.75)
 		(end 107.95 54.1)
@@
 	)
 	(segment
+		(start 116.9 69.87)
+		(end 116.92 69.85)
+		(width 1)
+		(layer "F.Cu")
+		(net 19)
+	)
+	(segment
+		(start 120.65 69.7)
+		(end 117.2 66.25)
+		(width 1)
+		(layer "F.Cu")
+		(net 19)
+	)
+	(segment
 		(start 111.32 57.47)
 		(end 126.21 57.47)
@@
 	)
 	(segment
-		(start 117.38 66.65)
-		(end 116.98 66.25)
+		(start 65.28 58.42)
+		(end 65.28 69.85)
 		(width 1)
 		(layer "F.Cu")
@@
 	)
 	(segment
-		(start 116.9 93.98)
-		(end 116.9 69.87)
+		(start 96.46 81.22)
+		(end 96.52 81.28)
 		(width 1)
 		(layer "F.Cu")
@@
 	)
 	(segment
-		(start 65.28 58.42)
-		(end 65.28 69.85)
+		(start 139.7 72.39)
+		(end 153.63 72.39)
 		(width 1)
 		(layer "F.Cu")
@@
 	)
 	(segment
-		(start 96.46 81.22)
-		(end 96.52 81.28)
+		(start 153.66 78.74)
+		(end 153.66 87.63)
 		(width 1)
 		(layer "F.Cu")
@@
 	)
 	(segment
-		(start 120.65 66.65)
-		(end 117.38 66.65)
+		(start 116.92 69.85)
+		(end 116.92 66.85)
 		(width 1)
 		(layer "F.Cu")
@@
 	)
 	(segment
-		(start 139.7 72.39)
-		(end 153.63 72.39)
+		(start 119.38 93.98)
+		(end 116.9 91.5)
 		(width 1)
 		(layer "F.Cu")
@@
 	)
 	(segment
-		(start 153.66 78.74)
-		(end 153.66 87.63)
+		(start 153.63 72.39)
+		(end 153.63 78.74)
 		(width 1)
 		(layer "F.Cu")
@@
 	)
 	(segment
-		(start 116.92 69.85)
-		(end 116.92 66.85)
+		(start 116.9 91.5)
+		(end 116.9 69.87)
 		(width 1)
 		(layer "F.Cu")
@@
 	)
 	(segment
-		(start 153.63 72.39)
-		(end 153.63 78.74)
+		(start 107.95 54.1)
+		(end 111 57.15)
 		(width 1)
 		(layer "F.Cu")
@@
 	)
 	(segment
-		(start 107.95 54.1)
-		(end 111 57.15)
+		(start 139.7 93.98)
+		(end 119.38 93.98)
 		(width 1)
 		(layer "F.Cu")
@@
 		(width 1)
 		(layer "F.Cu")
+		(net 19)
+	)
+	(segment
+		(start 117.2 66.25)
+		(end 116.98 66.25)
+		(width 1)
+		(layer "F.Cu")
