File: kicad/Projeto_led_natal/Projeto_led_natal-sem_led.kicad_sch (KiCad schematic)
At the start: 34 parts, among them P1 220K, Q1 BC548, Q2 BC548, Q3 BC548, Q4 BC548, T1 12+12 500mA

Commit message: from note-valmir
Other:
- title: Pisca de Natal - Sem Led -> (none)
- moved on the sheet: F1, SW1A, T1
Changed lines of the file:
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@@
 	(generator_version "8.0")
 	(paper "A4")
-	(title_block
-		(title "Pisca de Natal - Sem Led")
-	)
 	(junction
 		(at 92.71 98.425)
@@
 	(wire
 		(pts
-			(xy 103.505 56.515) (xy 103.505 66.675)
-		)
-		(stroke
-			(width 0)
-			(type default)
-		)
-	)
-	(wire
-		(pts
 			(xy 129.54 82.55) (xy 133.985 82.55)
 		)
@@
 	(wire
 		(pts
-			(xy 72.39 61.595) (xy 64.77 61.595)
+			(xy 79.375 61.595) (xy 71.755 61.595)
 		)
 		(stroke
@@
 	(wire
 		(pts
-			(xy 83.185 66.675) (xy 83.185 82.55)
+			(xy 83.185 65.405) (xy 83.185 82.55)
 		)
 		(stroke
@@
 	(wire
 		(pts
-			(xy 92.71 51.435) (xy 107.315 51.435)
+			(xy 99.695 51.435) (xy 107.315 51.435)
 		)
 		(stroke
@@
 	(wire
 		(pts
-			(xy 83.185 66.675) (xy 103.505 66.675)
+			(xy 83.185 65.405) (xy 106.68 65.405)
 		)
 		(stroke
@@
 	(wire
 		(pts
-			(xy 103.505 56.515) (xy 92.71 56.515)
-		)
-		(stroke
-			(width 0)
-			(type default)
-		)
-	)
-	(wire
-		(pts
 			(xy 149.225 86.995) (xy 149.225 98.425)
 		)
@@
 	(wire
 		(pts
-			(xy 69.215 51.435) (xy 72.39 51.435)
+			(xy 76.2 51.435) (xy 79.375 51.435)
 		)
 		(stroke
@@
 	(wire
 		(pts
+			(xy 99.695 56.515) (xy 106.68 56.515)
+		)
+		(stroke
+			(width 0)
+			(type default)
+		)
+	)
+	(wire
+		(pts
 			(xy 83.185 82.55) (xy 85.725 82.55)
 		)
@@
 	(wire
 		(pts
-			(xy 92.71 61.595) (xy 107.315 61.595)
+			(xy 99.695 61.595) (xy 107.315 61.595)
+		)
+		(stroke
+			(width 0)
+			(type default)
+		)
+	)
+	(wire
+		(pts
+			(xy 106.68 65.405) (xy 106.68 56.515)
 		)
 		(stroke
@@
 	(global_label "SA"
 		(shape input)
-		(at 92.71 61.595 0)
+		(at 99.695 61.595 0)
 		(effects
 			(font
@@
 		)
 		(property "Intersheetrefs" "${INTERSHEET_REFS}"
-			(at 92.71 61.595 0)
+			(at 99.695 61.595 0)
 			(effects
 				(font
@@
 	(global_label "AA"
 		(shape input)
-		(at 72.39 51.435 180)
+		(at 79.375 51.435 180)
 		(effects
 			(font
@@
 		)
 		(property "Intersheetrefs" "${INTERSHEET_REFS}"
-			(at 72.39 51.435 0)
+			(at 79.375 51.435 0)
 			(effects
 				(font
@@
 	(global_label "SB"
 		(shape input)
-		(at 92.71 51.435 0)
+		(at 99.695 51.435 0)
 		(effects
 			(font
@@
 		)
 		(property "Intersheetrefs" "${INTERSHEET_REFS}"
-			(at 92.71 51.435 0)
+			(at 99.695 51.435 0)
 			(effects
 				(font
@@
 	(global_label "AB"
 		(shape input)
-		(at 72.39 61.595 180)
+		(at 79.375 61.595 180)
 		(effects
 			(font
@@
 		)
 		(property "Intersheetrefs" "${INTERSHEET_REFS}"
-			(at 72.39 61.595 0)
+			(at 79.375 61.595 0)
 			(effects
 				(font
@@
 	(hierarchical_label "SB"
 		(shape input)
-		(at 92.71 51.435 0)
+		(at 99.695 51.435 0)
 		(fields_autoplaced yes)
 		(effects
@@
 	(symbol
 		(lib_id "Switch:SW_DPST_x2")
-		(at 64.135 51.435 0)
+		(at 71.12 51.435 0)
 		(unit 1)
 		(exclude_from_sim no)
@@
 		(fields_autoplaced yes)
 		(property "Reference" "SW1"
-			(at 64.135 47.625 0)
+			(at 71.12 47.625 0)
 			(effects
 				(font
@@
 		)
 		(property "Value" "~"
-			(at 64.135 47.625 0)
+			(at 71.12 47.625 0)
 			(effects
 				(font
@@
 		)
 		(property "Footprint" "Button_Switch_SMD:SW_DIP_SPSTx01_Slide_6.7x4.1mm_W6.73mm_P2.54mm_LowProfile_JPin"
-			(at 64.135 51.435 0)
+			(at 71.12 51.435 0)
 			(effects
 				(font
@@
 		)
 		(property "Datasheet" "~"
-			(at 64.135 51.435 0)
+			(at 71.12 51.435 0)
 			(effects
 				(font
@@
 		)
 		(property "Description" "Single Pole Single Throw (SPST) switch, separate symbol"
-			(at 64.135 51.435 0)
+			(at 71.12 51.435 0)
 			(effects
 				(font
@@
 	(symbol
 		(lib_id "Device:Fuse_Small")
-		(at 62.23 61.595 0)
+		(at 69.215 61.595 0)
 		(unit 1)
 		(exclude_from_sim no)
@@
 		(dnp no)
 		(property "Reference" "F1"
-			(at 62.23 56.515 0)
+			(at 69.215 56.515 0)
 			(effects
 				(font
@@
 		)
 		(property "Value" "500mA"
-			(at 62.23 59.055 0)
+			(at 69.215 59.055 0)
 			(effects
 				(font
@@
 		)
 		(property "Footprint" "Fuse:Fuse_1812_4532Metric"
-			(at 60.325 64.77 0)
+			(at 67.31 64.77 0)
 			(effects
 				(font
@@
 		)
 		(property "Datasheet" "~"
-			(at 62.23 61.595 0)
+			(at 69.215 61.595 0)
 			(effects
 				(font
@@
 		)
 		(property "Description" "Fuse, small symbol"
-			(at 62.23 61.595 0)
+			(at 69.215 61.595 0)
 			(effects
 				(font
@@
 	(symbol
 		(lib_id "Device:Transformer_1P_SS")
-		(at 82.55 56.515 0)
+		(at 89.535 56.515 0)
 		(unit 1)
 		(exclude_from_sim no)
@@
 		(fields_autoplaced yes)
 		(property "Reference" "T1"
-			(at 82.5627 46.355 0)
+			(at 89.5477 46.355 0)
 			(effects
 				(font
@@
 		)
 		(property "Value" "12+12 500mA"
-			(at 82.5627 48.895 0)
+			(at 89.5477 48.895 0)
 			(effects
 				(font
@@
 		)
 		(property "Footprint" "Transformer_SMD:Transformer_MACOM_SM-22"
-			(at 82.55 56.515 0)
+			(at 89.535 56.515 0)
 			(effects
 				(font
@@
 		)
 		(property "Datasheet" "~"
-			(at 82.55 56.515 0)
+			(at 89.535 56.515 0)
 			(effects
 				(font
@@
 		)
 		(property "Description" "Transformer, single primary, split secondary"
-			(at 82.55 56.515 0)
-			(effects
-				(font
+			(at 89.535 56.515 0)
+			(effects
+				(font
